Commit message: v2

File: description/robot_core.xacro (robot description, xacro)
@@ -1,4 +1,4 @@
 <?xml version="1.0"?>
-<robot name="robot" xmlns:xacro="http://ros.org/wiki/xacro">
+<robot xmlns:xacro="http://ros.org/wiki/xacro">
 <!-- Define robot constants -->
   <xacro:property name="base_width" value="0.241"/>
@@ -18,5 +18,5 @@
       </geometry>
       <material name="Cyan">
-        <color rgba="0 1.0 1.0 1.0"/>
+        <color rgba="0 1 1 1"/>
       </material>
     </visual>
@@ -55,5 +55,5 @@
         </geometry>
         <material name="red">
-        <color rgba=" 1 0 0 1" />
+          <color rgba=" 1 0 0 1" />
         </material>
     </visual>
@@ -66,5 +66,11 @@
  <!-- Wheels -->
   <xacro:macro name="wheel" params="prefix x_reflect y_reflect">
-    <link name="${prefix}_link">
+    <joint name="${prefix}_joint" type="continuous">
+      <parent link="base_link"/>
+      <child link="${prefix}"/>
+      <origin xyz="${x_reflect*wheel_front_xoff} ${y_reflect*(base_width/2+wheel_ygap)} ${-wheel_zoff}" rpy="0 0 0"/>
+      <axis xyz="0 1 0"/>
+    </joint>
+    <link name="${prefix}">
       <visual>
         <origin xyz="0 0 0" rpy="${pi/2} 0 0"/>
@@ -83,10 +89,4 @@
       </collision>
     </link>
-    <joint name="${prefix}_front_joint" type="continuous">
-      <parent link="base_link"/>
-      <child link="${prefix}_link"/>
-      <origin xyz="${x_reflect*wheel_front_xoff} ${y_reflect*(base_width/2+wheel_ygap)} ${-wheel_zoff}" rpy="0 0 0"/>
-      <axis xyz="0 1 0"/>
-    </joint>
   </xacro:macro>
   <xacro:wheel prefix="drivewhl_l_r" x_reflect="-1" y_reflect="1" />
