Commit message: v3

File: description/robot.urdf.xacro (robot description, xacro)
@@ -1,5 +1,5 @@
 <?xml version="1.0"?>
 <robot xmlns:xacro="http://www.ros.org/wiki/xacro"  name="robot">
-    <!-- Example link -->
-    <xacro:include filename="robot_core.xacro" />
+       <xacro:include filename="robot_core.xacro" />
+       <xacro:include filename="gazebo_control_diff.xacro" />
 </robot>

File: description/robot_core.xacro (robot description, xacro)
@@ -1,4 +1,5 @@
 <?xml version="1.0"?>
 <robot xmlns:xacro="http://ros.org/wiki/xacro">
+  <xacro:include filename="inertial_macros.xacro"/>
 <!-- Define robot constants -->
   <xacro:property name="base_width" value="0.241"/>
@@ -13,4 +14,12 @@
 <!-- Robot Base -->
   <link name="base_link">
+  </link>
+<!-- Robot Chassis-->
+ <joint name="chassis_joint" type="fixed">
+    <parent link="base_link"/>
+    <child link="chassis"/>
+    <origin xyz="0 0 0"/>
+  </joint>
+  <link name="chassis">
     <visual>
       <geometry>
@@ -26,5 +35,11 @@
       </geometry>
     </collision>
+    <xacro:inertial_box mass="3" x="${base_length}" y=" ${base_width}" z=" ${base_height}">
+      <origin xyz= "0 0 0" rpy="0 0 0"/>
+    </xacro:inertial_box>
   </link>
+  <gazebo reference="chassis">
+    <material>Gazebo/Blue</material>
+  </gazebo>
 <!-- Robot Footprint -->
   <link name="base_footprint"/>
@@ -51,10 +66,10 @@
     </visual>
     <visual>
-        <geometry>
-      <cylinder radius="0.0508" length="0.041"/>
-        </geometry>
-        <material name="red">
-          <color rgba=" 1 0 0 1" />
-        </material>
+      <geometry>
+        <cylinder radius="0.0508" length="0.041"/>
+      </geometry>
+      <material name="red">
+        <color rgba=" 1 0 0 1" />
+      </material>
     </visual>
     <collision>
@@ -63,5 +78,11 @@
       </geometry>
     </collision>
+    <xacro:inertial_cylinder mass="0.1" length="0.041" radius="0.0508">
+      <origin xyz="0 0 0.1" rpy="0 0 0"/>
+    </xacro:inertial_cylinder>
   </link>
+  <gazebo reference="laser_frame">
+    <material>Gazebo/Red</material>
+  </gazebo>
  <!-- Wheels -->
   <xacro:macro name="wheel" params="prefix x_reflect y_reflect">
@@ -88,5 +109,11 @@
         </geometry>
       </collision>
+      <xacro:inertial_cylinder mass="0.5" radius="${wheel_radius}" length="${wheel_width}">
+        <origin xyz="0 0 0.1" rpy="0 0 0"/>
+      </xacro:inertial_cylinder>
     </link>
+    <gazebo reference="${prefix}">
+      <material>Gazebo/Gray</material>
+    </gazebo>
   </xacro:macro>
   <xacro:wheel prefix="drivewhl_l_r" x_reflect="-1" y_reflect="1" />
