Commit message: v4

File: description/gazebo_control.xacro (robot description, xacro)
@@ -3,9 +3,12 @@
     <gazebo>
         <plugin name="diff_drive" filename="libgazebo_ros_diff_drive.so">
-            jackal_velocity_controller:
-  type: "diff_drive_controller/DiffDriveController"
-  left_wheel: ['front_left_wheel', 'rear_left_wheel']
-  right_wheel: ['front_right_wheel', 'rear_right_wheel']
-  publish_rate: 50
+            <!-- Wheel Information -->
+            <num_wheel_pairs>2</num_wheel_pairs>
+            <left_joint>drivewhl_l_f_joint</left_joint>
+            <left_joint>drivewhl_l_r_joint</left_joint>
+            <right_joint>drivewhl_r_f_joint</right_joint>
+            <right_joint>drivewhl_r_r_joint</right_joint>
+            <wheel_separation>0.35</wheel_separation>
+            <wheel_diameter>0.079</wheel_diameter>
             <!-- Limits -->
             <max_wheel_torque>200</max_wheel_torque>

File: description/robot.urdf.xacro (robot description, xacro)
@@ -2,4 +2,5 @@
 <robot xmlns:xacro="http://www.ros.org/wiki/xacro"  name="robot">
        <xacro:include filename="robot_core.xacro" />
-       <xacro:include filename="gazebo_control_diff.xacro" />
+       <xacro:include filename="gazebo_control.xacro" />
+       <xacro:include filename="lidar.xacro"/>
 </robot>

File: description/robot_core.xacro (robot description, xacro)
@@ -49,40 +49,4 @@
     <origin xyz="0.0 0.0 ${-(wheel_radius+wheel_zoff)}" rpy="0 0 0"/>
   </joint>
-<!-- LiDAR -->
- <joint name="laser_joint" type="fixed">
-     <parent link="base_link"/>
-     <child link="laser_frame"/>
-     <origin xyz="0 0 0.1" rpy="0 0 0"/>
-     <axis xyz="0 0 1" />
- </joint>
- <link name="laser_frame">
-	  <visual>
-	    <geometry>
-		    <cylinder radius="0.0508" length="0.041"/>
-	    </geometry>
-	    <material name="red">
-	    	<color rgba=" 1 0 0 1" />
-	    </material>
-    </visual>
-    <visual>
-      <geometry>
-        <cylinder radius="0.0508" length="0.041"/>
-      </geometry>
-      <material name="red">
-        <color rgba=" 1 0 0 1" />
-      </material>
-    </visual>
-    <collision>
-      <geometry>
-        <cylinder radius="0.0508" length="0.041"/>
-      </geometry>
-    </collision>
-    <xacro:inertial_cylinder mass="0.1" length="0.041" radius="0.0508">
-      <origin xyz="0 0 0.1" rpy="0 0 0"/>
-    </xacro:inertial_cylinder>
-  </link>
-  <gazebo reference="laser_frame">
-    <material>Gazebo/Red</material>
-  </gazebo>
  <!-- Wheels -->
   <xacro:macro name="wheel" params="prefix x_reflect y_reflect">
